File: pigmice-led-ring.sch (KiCad schematic (older format))
At the start: 34 parts, among them J1 +12V, J2 GND

Commit message: Add README, 22ohm -> 82ohm
Parts:
- R1, R2, R3, R4, R5, R6, R7, R8: value 22 -> 82
Changed lines of the file:
@@
 P 1500 1000
 F 0 "R1" H 1570 1046 50  0000 L CNN
-F 1 "22" H 1570 955 50  0000 L CNN
+F 1 "82" H 1570 955 50  0000 L CNN
 F 2 "Resistor_SMD:R_0805_2012Metric_Pad1.15x1.40mm_HandSolder" V 1430 1000 50  0001 C CNN
 F 3 "~" H 1500 1000 50  0001 C CNN
@@
 P 1900 1000
 F 0 "R2" H 1970 1046 50  0000 L CNN
-F 1 "22" H 1970 955 50  0000 L CNN
+F 1 "82" H 1970 955 50  0000 L CNN
 F 2 "Resistor_SMD:R_0805_2012Metric_Pad1.15x1.40mm_HandSolder" V 1830 1000 50  0001 C CNN
 F 3 "~" H 1900 1000 50  0001 C CNN
@@
 P 2250 1000
 F 0 "R3" H 2320 1046 50  0000 L CNN
-F 1 "22" H 2320 955 50  0000 L CNN
+F 1 "82" H 2320 955 50  0000 L CNN
 F 2 "Resistor_SMD:R_0805_2012Metric_Pad1.15x1.40mm_HandSolder" V 2180 1000 50  0001 C CNN
 F 3 "~" H 2250 1000 50  0001 C CNN
@@
 P 2650 1000
 F 0 "R4" H 2720 1046 50  0000 L CNN
-F 1 "22" H 2720 955 50  0000 L CNN
+F 1 "82" H 2720 955 50  0000 L CNN
 F 2 "Resistor_SMD:R_0805_2012Metric_Pad1.15x1.40mm_HandSolder" V 2580 1000 50  0001 C CNN
 F 3 "~" H 2650 1000 50  0001 C CNN
@@
 P 3000 1000
 F 0 "R5" H 3070 1046 50  0000 L CNN
-F 1 "22" H 3070 955 50  0000 L CNN
+F 1 "82" H 3070 955 50  0000 L CNN
 F 2 "Resistor_SMD:R_0805_2012Metric_Pad1.15x1.40mm_HandSolder" V 2930 1000 50  0001 C CNN
 F 3 "~" H 3000 1000 50  0001 C CNN
@@
 P 3400 1000
 F 0 "R6" H 3470 1046 50  0000 L CNN
-F 1 "22" H 3470 955 50  0000 L CNN
+F 1 "82" H 3470 955 50  0000 L CNN
 F 2 "Resistor_SMD:R_0805_2012Metric_Pad1.15x1.40mm_HandSolder" V 3330 1000 50  0001 C CNN
 F 3 "~" H 3400 1000 50  0001 C CNN
@@
 P 3750 1000
 F 0 "R7" H 3820 1046 50  0000 L CNN
-F 1 "22" H 3820 955 50  0000 L CNN
+F 1 "82" H 3820 955 50  0000 L CNN
 F 2 "Resistor_SMD:R_0805_2012Metric_Pad1.15x1.40mm_HandSolder" V 3680 1000 50  0001 C CNN
 F 3 "~" H 3750 1000 50  0001 C CNN
@@
 P 4150 1000
 F 0 "R8" H 4220 1046 50  0000 L CNN
-F 1 "22" H 4220 955 50  0000 L CNN
+F 1 "82" H 4220 955 50  0000 L CNN
 F 2 "Resistor_SMD:R_0805_2012Metric_Pad1.15x1.40mm_HandSolder" V 4080 1000 50  0001 C CNN
 F 3 "~" H 4150 1000 50  0001 C CNN
