File: pigmice-led-ring.kicad_pcb (KiCad board)
At the start: 2 copper layers, 46 x 51 mm, 47 parts, among them J1 Conn_01x02_Female, J2 Conn_01x03_Female, U1 LMR62014XMF

Commit message: Remove photos, text
Parts:
- removed G***: LOGO, led-ring:logo
- removed the REF** at (76.5, 60.5)
Other:
- board text removed: "github.com/Pigmice2733/led-ring v0.3.6"

Commit message: Add CERN OHL v2 permissive license
Other:
- board text added: "Licensed under CERN-OHL-P v2"
Changed lines of the file:
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@@
-(kicad_pcb (version 20171130) (host pcbnew 5.1.5-52549c5~84~ubuntu19.04.1)
+(kicad_pcb (version 20171130) (host pcbnew 5.1.5-52549c5~86~ubuntu19.04.1)
   (general
     (thickness 1.6)
-    (drawings 13)
+    (drawings 14)
     (tracks 136)
     (zones 0)
@@
     )
   )
+  (gr_text "Licensed under CERN-OHL-P v2" (at 90 64.2) (layer B.SilkS)
+    (effects (font (size 1.5 1.5) (thickness 0.3)) (justify mirror))
+  )
   (gr_circle (center 90 80) (end 103.5 80) (layer Edge.Cuts) (width 0.15))
